File: soundrocket/soundrocket.kicad_pcb (KiCad board)
At the start: 2 copper layers, 1 part

Commit message: work
Parts:
- added REF**: XFMR_PE-65612NL, PE_65612NL:XFMR_PE-65612NL, F.Cu at (223.8, 91.3)
- added REF**: SOP65P640X120-28N, DIT4192IPW:SOP65P640X120-28N, F.Cu at (182.6, 91.3)
- moved REF** 0.79 mm to (245.7, 87.5)
Routing:
- net (no net): track 0.00 -> 34.7 mm

Commit message: schematic start
Parts:
- removed REF**: XFMR_PE-65612NL, PE_65612NL:XFMR_PE-65612NL
- removed REF**: Jack_XLR_Neutrik_NC3FAAH1-DA_Horizontal, Connector_Audio:Jack_XLR_Neutrik_NC3FAAH1-DA_Horizontal
- removed REF**: SOP65P640X120-28N, DIT4192IPW:SOP65P640X120-28N
- added J1: XLR3 MALE (OUT), Connector_Audio:Jack_XLR_Neutrik_NC3FAAH-0_Horizontal, F.Cu at (203.0, 35.1)
- added SW1: SW_Push, Button_Switch_THT:SW_PUSH-12mm, F.Cu at (131.9, 69.5)
- added SW2: RotaryEncoder_Switch, Rotary_Encoder:RotaryEncoder_Bourns_Vertical_PEC12R-3x17F-Sxxxx, F.Cu at (160.7, 66.0)
- added U1: Teensy4.0, KiCad Models:Teensy40, F.Cu at (143.5, 39.9)
- added U2: DIT4192IPW, DIT4192IPW:SOP65P640X120-28N, F.Cu at (171.2, 39.7)
Routing:
- net Net-(U1-0_RX1_CRX2_CS1): track 0.00 -> 48.7 mm, vias 0 -> 2
- net /DIT4192-TX-: track 0.00 -> 43.1 mm
- net /DIT4192-TX+: track 0.00 -> 43.1 mm
- net Net-(U1-7_RX2_OUT1A): track 0.00 -> 36.1 mm, vias 0 -> 2
- net Net-(U1-6_OUT1D): track 0.00 -> 35.2 mm
- net Net-(U1-5_IN2): track 0.00 -> 35.1 mm
- net (no net): track 34.7 -> 0.00 mm
- net Net-(U1-11_MOSI_CTX1): track 0.00 -> 29.4 mm
- net Net-(U1-10_CS_MQSR): track 0.00 -> 28.3 mm, vias 0 -> 2
- net GND: track 0.00 -> 20.4 mm, vias 0 -> 3
- net Net-(U1-3_LRCLK2): track 0.00 -> 17.2 mm
- net Net-(U1-2_OUT2): track 0.00 -> 10.4 mm
- added copper zone on In2.Cu, net GND
Other:
- copper layers 2 -> 4

Commit message: Getting close to final
Parts:
- added 5V: 5V, TestPoint:TestPoint_THTPad_D1.5mm_Drill0.7mm, F.Cu at (121.9, 48.3)
- added C1: C_Small, KiCad Models:CAPRR254W54L381T254H466, F.Cu at (165.1, 67.3)
- added C2: C_Small, KiCad Models:CAPRR254W54L381T254H466, F.Cu at (165.1, 62.2)
- added GND: GND, TestPoint:TestPoint_THTPad_D1.5mm_Drill0.7mm, F.Cu at (121.9, 53.3)
- added T1: PE-65612NL, PE_65612NL:XFMR_PE-65612NL, F.Cu at (179.8, 50.8)
- moved J1 13.7 mm to (196.4, 47.0)
Connections:
- J1 pad 1: /DIT4192-TX+ -> /XLR-TX+
- J1 pad 2: /DIT4192-TX- -> /XLR-TX-
- U1 pad 1: GND -> unconnected-(U1-GND-Pad1)
- U1 pad 33: GND -> 5V0
- U2 pad 19: GND -> 5V0
Routing:
- net Net-(U2-V_IO): track 0.00 -> 48.5 mm
- net Net-(U1-23_A9_CRX1_MCLK1): track 0.00 -> 44.0 mm, vias 0 -> 1
- net Net-(U1-21_A7_RX5_BCLK1): track 0.00 -> 38.0 mm
- net Net-(U1-19_A5_SCL0): track 0.00 -> 34.4 mm, vias 0 -> 1
- net Net-(U1-20_A6_TX5_LRCLK1): track 0.00 -> 33.5 mm
- net /DIT4192-TX+: track 43.1 -> 12.5 mm
- net /DIT4192-TX-: track 43.1 -> 13.5 mm
- net /XLR-TX+: track 0.00 -> 12.0 mm
- net /XLR-TX-: track 0.00 -> 11.3 mm
- net Net-(U1-6_OUT1D): track 35.2 -> 44.2 mm
- net GND: track 20.4 -> 15.7 mm
- net Net-(U1-5_IN2): track 35.1 -> 39.4 mm
- net 5V0: track 0.00 -> 2.60 mm, vias 0 -> 1
- net Net-(U1-0_RX1_CRX2_CS1): track 48.7 -> 49.3 mm, vias 2 -> 1
- net Net-(U1-10_CS_MQSR): track 28.3 -> 27.7 mm, vias 2 -> 1
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- added copper zone on In1.Cu, net 5V0
Other:
- board outline added: 92.7 x 45.7 mm
- board text added: "Design by Daniel Anderson"

Commit message: Removed /5V0 net
Parts:
- added C3: C_Small, KiCad Models:CAPRR254W54L381T254H466, F.Cu at (123.2, 61.2)
- added C4: C_Small, KiCad Models:CAPRR254W54L381T254H466, F.Cu at (144.0, 69.8)
Connections:
- SW1 pad 1: GND -> Net-(C3-Pad1)
- SW2 pad S1: GND -> Net-(C4-Pad1)
Routing:
- net Net-(C3-Pad1): track 0.00 -> 9.90 mm
- net Net-(C4-Pad1): track 0.00 -> 3.47 mm

Commit message: soundbullet format
Parts:
- removed J1: XLR3 MALE (OUT), Connector_Audio:Jack_XLR_Neutrik_NC3FAAH-0_Horizontal
- removed SW1: SW_Push, Button_Switch_THT:SW_PUSH-12mm
- removed SW2: RotaryEncoder_Switch, Rotary_Encoder:RotaryEncoder_Bourns_Vertical_PEC12R-3x17F-Sxxxx
- added ?: , , F.Cu at (175.3, 66.3)
- added ?: , , F.Cu at (175.3, 63.5)
- added REF**: TestPoint_THTPad_D1.5mm_Drill0.7mm, TestPoint:TestPoint_THTPad_D1.5mm_Drill0.7mm, F.Cu at (160.0, 53.3)
- added REF**: TestPoint_THTPad_D1.5mm_Drill0.7mm, TestPoint:TestPoint_THTPad_D1.5mm_Drill0.7mm, F.Cu at (154.9, 53.3)
- added SW1+: TestPoint_THTPad_D1.5mm_Drill0.7mm, TestPoint:TestPoint_THTPad_D1.5mm_Drill0.7mm, F.Cu at (134.6, 51.8)
- added SW1-: TestPoint_THTPad_D1.5mm_Drill0.7mm, TestPoint:TestPoint_THTPad_D1.5mm_Drill0.7mm, F.Cu at (129.3, 51.8)
- added SW2+: TestPoint_THTPad_D1.5mm_Drill0.7mm, TestPoint:TestPoint_THTPad_D1.5mm_Drill0.7mm, F.Cu at (139.7, 51.8)
- added SW2-: TestPoint_THTPad_D1.5mm_Drill0.7mm, TestPoint:TestPoint_THTPad_D1.5mm_Drill0.7mm, F.Cu at (144.8, 51.8)
- moved C4 17.8 mm to (149.9, 53.1)
- moved 5V 16.1 mm to (124.0, 32.3)
- moved C3 8.23 mm to (124.5, 53.1)
- moved C2 8.03 mm to (157.5, 59.7), turned to 90 degrees
- moved C1 8.03 mm to (162.6, 59.7), turned to 90 degrees
- moved T1 7.16 mm to (173.5, 54.1), turned to -90 degrees
- moved GND 6.19 mm to (124.0, 47.5)
Routing:
- net Net-(U1-6_OUT1D): track 44.2 -> 17.7 mm
- net Net-(U1-5_IN2): track 39.4 -> 15.1 mm
- net Net-(U1-3_LRCLK2): track 17.2 -> 5.37 mm
- net Net-(U1-2_OUT2): track 10.4 -> 4.32 mm
- net Net-(C3-Pad1): track 9.90 -> 4.83 mm
- net /DIT4192-TX-: track 13.5 -> 9.82 mm
- net /XLR-TX+: track 12.0 -> 8.68 mm
- net Net-(U1-0_RX1_CRX2_CS1): track 49.3 -> 46.7 mm
- net /XLR-TX-: track 11.3 -> 9.35 mm
- net /DIT4192-TX+: track 12.5 -> 10.6 mm
- net Net-(C4-Pad1): track 3.47 -> 5.08 mm
- net Net-(U2-V_IO): track 48.5 -> 47.7 mm
- net Net-(U1-21_A7_RX5_BCLK1): track 38.0 -> 37.4 mm
- net Net-(U1-7_RX2_OUT1A): track 36.1 -> 35.5 mm
Other:
- board size 92.7 x 45.7 mm -> 58.2 x 43.9 mm
- board text added: "Designed by Dan A"
- board text added: "TX+"
- board text added: "TX-"
- board text removed: "Design by Daniel Anderson"

Commit message: compact version complete
Parts:
- removed REF** (x2), SW1+, SW2+: TestPoint_THTPad_D1.5mm_Drill0.7mm, TestPoint:TestPoint_THTPad_D1.5mm_Drill0.7mm
- moved ? 21.3 mm to (157.5, 54.6), turned to -90 degrees
- moved ? 15.9 mm to (162.1, 54.6), turned to -90 degrees
- moved C1 11.4 mm to (153.7, 52.6), turned to -90 degrees
- moved C2 11.4 mm to (148.6, 52.6), turned to -90 degrees
- moved C4 8.48 mm to (141.5, 51.8), turned to 0 degrees
- moved SW2- 7.62 mm to (137.2, 51.8)
- moved T1 5.48 mm to (172.2, 48.8)
- moved U2 3.62 mm to (171.2, 36.1)
- moved C3 3.54 mm to (127.8, 51.8), turned to 180 degrees
- moved SW1- 2.79 mm to (132.1, 51.8)
Routing:
- net Net-(U1-6_OUT1D): track 17.7 -> 10.5 mm
- net Net-(U1-5_IN2): track 15.1 -> 7.93 mm
- net /XLR-TX+: track 8.68 -> 14.1 mm
- net Net-(U1-3_LRCLK2): track 5.37 -> 0.00 mm
- net /XLR-TX-: track 9.35 -> 14.2 mm
- net Net-(U1-2_OUT2): track 4.32 -> 0.00 mm
- net Net-(U1-7_RX2_OUT1A): track 35.5 -> 39.6 mm
- net Net-(U1-21_A7_RX5_BCLK1): track 37.4 -> 33.5 mm
- net Net-(U2-V_IO): track 47.7 -> 44.1 mm
- net Net-(U1-20_A6_TX5_LRCLK1): track 33.1 -> 29.5 mm
- net Net-(U1-10_CS_MQSR): track 27.7 -> 31.0 mm
- net GND: track 15.7 -> 18.4 mm
- net /DIT4192-TX+: track 10.6 -> 8.40 mm
- net Net-(U1-0_RX1_CRX2_CS1): track 46.7 -> 48.9 mm
- net 5V0: track 2.60 -> 4.70 mm
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Other:
- board size 58.2 x 43.9 mm -> 58.2 x 28.4 mm
- board text added: "EA"
- board text added: "EB"
- board text added: "SW1"
- board text added: "SW2"

Commit message: Update soundrocket.kicad_pcb
Routing:
- net GND: track 18.4 -> 11.8 mm
Changed lines of the file:
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@@
-	)
-	(segment
-		(start 174.79 40.17)
-		(end 175.006 40.386)
-		(width 0.25)
-		(layer "F.Cu")
-		(net 6)
 	)
 	(segment
@@
 	)
 	(segment
-		(start 176.53 40.386)
-		(end 177.8 39.116)
+		(start 173.49 39.886)
+		(end 174.752 41.148)
 		(width 0.25)
 		(layer "F.Cu")
@@
 	)
 	(segment
-		(start 173.49 39.722999)
-		(end 174.661001 40.894)
+		(start 174.79 41.11)
+		(end 174.752 41.148)
 		(width 0.25)
 		(layer "F.Cu")
@@
 	)
 	(segment
-		(start 173.49 38.938)
-		(end 173.49 39.722999)
-		(width 0.25)
-		(layer "F.Cu")
-		(net 6)
-	)
-	(segment
-		(start 177.8 39.878)
-		(end 177.8 39.116)
+		(start 175.44 38.938)
+		(end 175.44 40.46)
 		(width 0.25)
 		(layer "F.Cu")
@@
 	(segment
 		(start 174.79 38.938)
-		(end 174.79 40.17)
-		(width 0.25)
-		(layer "F.Cu")
-		(net 6)
-	)
-	(segment
-		(start 175.006 40.386)
-		(end 176.53 40.386)
+		(end 174.79 41.11)
 		(width 0.25)
 		(layer "F.Cu")
@@
 	)
 	(segment
-		(start 175.44 38.938)
-		(end 177.622 38.938)
+		(start 175.44 40.46)
+		(end 174.752 41.148)
 		(width 0.25)
 		(layer "F.Cu")
@@
 	)
 	(segment
-		(start 176.784 40.894)
-		(end 177.8 39.878)
-		(width 0.25)
-		(layer "F.Cu")
-		(net 6)
-	)
-	(segment
-		(start 177.622 38.938)
-		(end 177.8 39.116)
-		(width 0.25)
-		(layer "F.Cu")
-		(net 6)
-	)
-	(segment
-		(start 174.661001 40.894)
-		(end 176.784 40.894)
+		(start 173.49 38.938)
+		(end 173.49 39.886)
 		(width 0.25)
 		(layer "F.Cu")
@@
 	)
 	(via
-		(at 177.8 39.116)
+		(at 174.752 41.148)
 		(size 0.8)
 		(drill 0.4)

Commit message: Gerbers
Parts:
- moved C4 1.98 mm to (140.2, 53.3)
- moved SW1- 1.98 mm to (130.8, 53.3)
- moved SW2- 1.98 mm to (135.9, 53.3)
- moved C3 1.98 mm to (126.5, 53.3)
- moved C2 1.63 mm to (147.3, 53.6)
- moved C1 1.63 mm to (152.4, 53.6)
Routing:
- net Net-(U1-5_IN2): track 7.93 -> 7.08 mm
- net Net-(U1-6_OUT1D): track 10.5 -> 9.62 mm
Changed lines of the file:
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@@
 			(outputformat 1)
 			(mirror no)
-			(drillshape 1)
+			(drillshape 0)
 			(scaleselection 1)
 			(outputdirectory "")
@@
 	(footprint "KiCad Models:CAPRR254W54L381T254H466"
 		(layer "F.Cu")
-		(at 148.59 52.578 -90)
+		(at 147.32 53.594 -90)
 		(property "Reference" "C2"
 			(at 2.794 0 180)
@@
 	(footprint "KiCad Models:CAPRR254W54L381T254H466"
 		(layer "F.Cu")
-		(at 141.478 51.816)
+		(at 140.208 53.34)
 		(property "Reference" "C4"
 			(at 2.794 0 90)
@@
 	(footprint "TestPoint:TestPoint_THTPad_D1.5mm_Drill0.7mm"
 		(layer "F.Cu")
-		(at 137.16 51.816)
+		(at 135.89 53.34)
 		(descr "THT pad as test Point, diameter 1.5mm, hole diameter 0.7mm")
 		(tags "test point THT pad")
@@
 	(footprint "TestPoint:TestPoint_THTPad_D1.5mm_Drill0.7mm"
 		(layer "F.Cu")
-		(at 132.08 51.816)
+		(at 130.81 53.34)
 		(descr "THT pad as test Point, diameter 1.5mm, hole diameter 0.7mm")
 		(tags "test point THT pad")
@@
 	(footprint "KiCad Models:CAPRR254W54L381T254H466"
 		(layer "F.Cu")
-		(at 153.67 52.578 -90)
+		(at 152.4 53.594 -90)
 		(property "Reference" "C1"
 			(at 2.794 0 0)
@@
 	(footprint "KiCad Models:CAPRR254W54L381T254H466"
 		(layer "F.Cu")
-		(at 127.762 51.816 180)
+		(at 126.492 53.34 180)
 		(property "Reference" "C3"
 			(at 2.794 0 90)
@@
 	)
 	(gr_text "Designed by Dan A"
-		(at 121.666 56.642 0)
+		(at 178.816 57.15 90)
 		(layer "F.SilkS")
 		(effects
 			(font
-				(size 1 1)
-				(thickness 0.2)
+				(size 0.8 0.8)
+				(thickness 0.16)
 				(bold yes)
 			)
@@
 	)
 	(segment
-		(start 142.24 47.498)
-		(end 146.05 51.308)
+		(start 147.066 52.324)
+		(end 147.32 52.324)
 		(width 0.25)
 		(layer "F.Cu")
@@
 	)
 	(segment
-		(start 146.05 51.308)
-		(end 148.59 51.308)
+		(start 142.24 47.498)
+		(end 147.066 52.324)
 		(width 0.25)
 		(layer "F.Cu")
@@
 	)
 	(segment
-		(start 151.638 49.276)
-		(end 153.67 51.308)
+		(start 144.78 47.498)
+		(end 148.082 50.8)
 		(width 0.25)
 		(layer "F.Cu")
@@
 	)
 	(segment
-		(start 146.558 49.276)
-		(end 151.638 49.276)
+		(start 148.082 50.8)
+		(end 150.876 50.8)
 		(width 0.25)
 		(layer "F.Cu")
@@
 	)
 	(segment
-		(start 144.78 47.498)
-		(end 146.558 49.276)
+		(start 150.876 50.8)
+		(end 152.4 52.324)
 		(width 0.25)
 		(layer "F.Cu")
@@
 	)
 	(segment
-		(start 132.08 51.816)
-		(end 129.032 51.816)
+		(start 130.81 53.34)
+		(end 127.762 53.34)
 		(width 0.25)
 		(layer "F.Cu")
@@
 	)
 	(segment
-		(start 140.208 51.816)
-		(end 137.16 51.816)
+		(start 138.938 53.34)
+		(end 135.89 53.34)
 		(width 0.25)
 		(layer "F.Cu")
