File: soundrocket/soundrocket.kicad_pcb (KiCad board)
At the start: 4 copper layers, 85.3 x 45.7 mm, 12 parts, among them J1 XLR3 MALE (OUT), SW1 SW_Push, SW2 RotaryEncoder_Switch, T1 PE-65612NL, U1 Teensy4.0, U2 DIT4192IPW

Commit message: Gerbers
Parts:
- moved T1 21.9 mm to (192.8, 64.5), turned to 0 degrees
- moved 5V 16.0 mm to (121.9, 32.3)
- moved C1 9.65 mm to (174.8, 67.3)
- moved C2 9.65 mm to (174.8, 62.2)
- moved J1 9.40 mm to (188.5, 37.6)
- moved SW2 7.87 mm to (168.5, 66.0)
- moved C4 5.84 mm to (149.9, 69.8)
- moved GND 5.84 mm to (121.9, 47.5)
- moved SW1 1.52 mm to (133.4, 69.5)
Routing:
- net /XLR-TX-: track 30.4 -> 59.4 mm
- net /XLR-TX+: track 30.3 -> 58.1 mm
- net /DIT4192-TX-: track 9.82 -> 33.2 mm
- net /DIT4192-TX+: track 10.6 -> 32.0 mm
- net Net-(U1-5_IN2): track 39.4 -> 49.2 mm
- net Net-(U1-6_OUT1D): track 44.2 -> 52.5 mm
- net Net-(U1-3_LRCLK2): track 17.2 -> 22.5 mm
- net Net-(C4-Pad1): track 3.47 -> 5.25 mm
- net Net-(C3-Pad1): track 9.90 -> 11.4 mm
- net Net-(U1-2_OUT2): track 10.4 -> 11.1 mm

Commit message: Hardware Test & Revision 2
Parts:
- added R1: R_Small (10k), KiCad Models:STA_CF14_STP, F.Cu at (165.6, 71.4)
- added R2: R_Small (10k), KiCad Models:STA_CF14_STP, F.Cu at (165.6, 67.3)
- added R3: R_Small (10k), KiCad Models:STA_CF14_STP, F.Cu at (167.6, 52.7)
- added R4: R_Small (10k), KiCad Models:STA_CF14_STP, F.Cu at (172.0, 52.7)
- added R5: R_Small, KiCad Models:STA_CF14_STP, F.Cu at (122.4, 51.3)
- J1: footprint Connector_Audio:Jack_XLR_Neutrik_NC3FAAH-0_Horizontal -> Connector_Audio:Jack_XLR_Neutrik_NC3MAAV_Vertical
- moved C4 34.9 mm to (141.0, 53.3), turned to 180 degrees
- moved C3 31.9 mm to (146.1, 53.3), turned to 0 degrees
- moved C1 12.6 mm to (131.8, 52.1), turned to 90 degrees
- moved C2 12.4 mm to (143.5, 59.2)
- moved SW2 6.35 mm to (162.2, 66.0)
- moved J1 4.38 mm to (187.2, 41.8)
- moved SW1 4.02 mm to (129.4, 69.5)
- renumbered C3 to C1, C4 to C2, C1 to C3, C2 to C4
Connections:
- net Net-(U2-V_IO) renamed 3V3
- C1 pad 1: Net-(C3-Pad1) -> Net-(U1-2_OUT2)
- C2 pad 1: Net-(C4-Pad1) -> Net-(U1-3_LRCLK2)
- SW1 pad 1: Net-(C3-Pad1) -> GND
- SW2 pad A: Net-(U1-6_OUT1D) -> Net-(R1-Pad1)
- SW2 pad B: Net-(U1-5_IN2) -> Net-(R2-Pad1)
- SW2 pad S1: Net-(C4-Pad1) -> GND
Routing:
- net 3V3: track 48.5 -> 159.1 mm
- net /XLR-TX-: track 59.4 -> 40.6 mm
- net /XLR-TX+: track 58.1 -> 39.9 mm
- net Net-(R1-Pad1): track 0.00 -> 17.0 mm
- net Net-(U1-6_OUT1D): track 52.5 -> 36.9 mm
- net Net-(U1-5_IN2): track 49.2 -> 34.5 mm
- net Net-(R2-Pad1): track 0.00 -> 13.9 mm
- net Net-(U1-2_OUT2): track 11.1 -> 22.5 mm
- net Net-(C3-Pad1): track 11.4 -> 0.00 mm
- net Net-(C4-Pad1): track 5.25 -> 0.00 mm
- net Net-(U1-0_RX1_CRX2_CS1): track 49.3 -> 46.3 mm
- net Net-(U1-3_LRCLK2): track 22.5 -> 20.0 mm
- net Net-(U1-23_A9_CRX1_MCLK1): track 44.0 -> 44.6 mm
Other:
- board text added: "Designed by Daniel A."
- board text added: "TX+"
- board text added: "TX-"
- board text removed: "Design by Daniel Anderson"
